Commit message: up to date

File: Robot_1/urdf/Robot_1.urdf (robot description, URDF)
Before this commit: robot Robot_1, 4 links, 3 joints
Joints:
- joint elevator: origin xyz=0 -0.4825 0.6682 rpy=1.5708 0 0 -> xyz=0.4825 0 0.6682 rpy=3.141628 -1.5708 0
- joint wheel_left: axis 0 0 0 -> 1 0 0; origin xyz=0.181 -0.42691 0.0733 rpy=0 1.4923 1.5708 -> xyz=0.42691 0.23 0.0733 rpy=-1.4923 0 1.5708
- joint wheel_right: axis 0 0 0 -> -1 0 0; origin xyz=-0.23 -0.42691 0.0733 rpy=2.7865 0 3.1416 -> xyz=0.42691 -0.23 0.0733 rpy=2.7865 0 -1.5708

File: infi_sim_v1/models/OPTIMUS_robot_001/model.xacro (robot description, xacro)
@@ -7,11 +7,11 @@
     <xacro:property name="MANIPULATOR_MOUNT_Z" value="0.0"/>
     <xacro:include filename="manipulator_h.xacro"/>
-    <xacro:include filename="sensors/xtion_pro_live.urdf.xacro"/>
-    <xacro:xtion_pro_live name="rgbd_camera" parent="end">
-        <origin xyz="0 0 0.1" rpy="0 0 0"/>
-        <origin xyz="0 0 0.1" rpy="${-90.0 * deg_to_rad} 0 ${-90.0 * deg_to_rad}"/>
+    <!--xacro:include filename="sensors/xtion_pro_live.urdf.xacro"/-->
+    <!--xacro:xtion_pro_live name="rgbd_camera" parent="end">
+        <origin xyz="0 0 0.1" rpy="0 0 0"/-->
+        <!--origin xyz="0 0 0.1" rpy="${-90.0 * deg_to_rad} 0 ${-90.0 * deg_to_rad}"/-->
         <!--<origin xyz="0 0 0.1" rpy="0 ${75.0 * deg_to_rad} 0"/>-->
         <!--<optical_origin xyz="0 0 0.1" rpy="${-90.0 * deg_to_rad} 0 ${-90.0 * deg_to_rad}"/>-->
-    </xacro:xtion_pro_live>
+    <!--/xacro:xtion_pro_live-->
     <xacro:property name="INTEL_D435_MOUNT_LINK" value="camera_mount_dummy_link"/>
     <xacro:property name="INTEL_D435_MOUNT_X" value="0.1"/>
@@ -215,4 +215,5 @@
     <!-- Elevator -->
     <joint name="j_elev" type="prismatic">
+    <!--joint name="j_elev" type="fixed"-->
         <parent link="base_link"/>
         <child link="elevator"/>
@@ -245,5 +246,5 @@
     </link>
     <!-- Sensors -->
-    <joint name="j_ray_sensor_back" type="fixed">
+    <!--joint name="j_ray_sensor_back" type="fixed">
         <parent link="base_link"/>
         <child link="ray_sensor_back"/>
@@ -292,5 +293,5 @@
             </plugin>
         </sensor>
-    </gazebo>
+    </gazebo-->
     <joint name="j_ray_sensor_front" type="fixed">
         <parent link="base_link"/>
@@ -336,5 +337,5 @@
                 <topicName>/scan</topicName>
                 <frameName>ray_sensor_front</frameName>
-                <ns>/optimus</ns>
+                <!--ns>/optimus</ns-->
                 <hokuyoMinIntensity>101</hokuyoMinIntensity>
             </plugin>
@@ -440,5 +441,5 @@
         </plugin>
         <plugin name="optimus_diff_drive" filename="libgazebo_ros_diff_drive.so">
-            <commandTopic>/optimus/cmd_vel</commandTopic>
+            <commandTopic>cmd_vel</commandTopic>
             <odometryTopic>odom</odometryTopic>
             <odometryFrame>odom</odometryFrame>
@@ -459,10 +460,10 @@
             <rosDebugLevel>na</rosDebugLevel>
         </plugin>
-        <plugin name="joint_state_publisher" filename="libgazebo_ros_joint_state_publisher.so">
+        <!--plugin name="joint_state_publisher" filename="libgazebo_ros_joint_state_publisher.so">
             <robotNamespace></robotNamespace>
             <jointName>j_elev, joint1, joint2, joint3, joint4, joint5, joint6</jointName>
             <updateRate>100.0</updateRate>
             <alwaysOn>true</alwaysOn>
-        </plugin>
+        </plugin-->
     </gazebo>
 </robot>
