Commit message: up to date

File: infi_sim_v1/models/OPTIMUS_robot_001/model.xacro (robot description, xacro)
@@ -2,4 +2,5 @@
     <xacro:property name="M_PI" value="3.1415926535897931"/>
     <xacro:property name="deg_to_rad" value="0.01745329251994329577"/>
+    <xacro:property name="camera_link" value="0.05" /> <!-- Size of square 'camera' box -->
     <xacro:property name="MANIPULATOR_MOUNT_LINK" value="elevator"/>
     <xacro:property name="MANIPULATOR_MOUNT_X" value="0.04"/>
@@ -18,7 +19,7 @@
     <xacro:property name="INTEL_D435_MOUNT_Y" value="-0.045"/>
     <xacro:property name="INTEL_D435_MOUNT_Z" value="0.1"/>
-    <xacro:property name="INTEL_D435_MOUNT_R" value="0"/>
-    <xacro:property name="INTEL_D435_MOUNT_P" value="0"/>
-    <xacro:property name="INTEL_D435_MOUNT_Y" value="0"/>
+    <xacro:property name="INTEL_D435_MOUNT_R" value="${M_PI*0.0}"/>
+    <xacro:property name="INTEL_D435_MOUNT_P" value="${M_PI*0.0}"/>
+    <xacro:property name="INTEL_D435_MOUNT_Y" value="${M_PI*0.0}"/>
     <!--<xacro:include filename="sensors/intel_d435.xacro"/>-->
     <!--    <xacro:include filename="sensors/intel_cam.xacro" name="camera_link" ros_topic="/d435"/>-->
