Commit message: working depth_cam

File: infi_sim_v1/models/OPTIMUS_robot_001/model-no-arm.xacro (robot description, xacro)
@@ -15,5 +15,5 @@
     <xacro:property name="INTEL_D435_MOUNT_P" value="${M_PI*0.0}"/>
     <xacro:property name="INTEL_D435_MOUNT_Y" value="${M_PI*0.0}"/>
-    <!--xacro:include filename="sensors/intel_d435.xacro"/-->
+    <xacro:include filename="sensors/intel_d435.xacro"/>
     <!--xacro:include filename="sensors/intel_cam.xacro" name="camera_link" ros_topic="/d435"/-->
     <link name="base_footprint"/>

File: infi_sim_v1/models/OPTIMUS_robot_001/sensors/intel_d435.xacro (robot description, xacro)
@@ -1,4 +1,24 @@
 <?xml version="1.0"?>
 <robot name="intel_d435" xmlns:xacro="http://www.ros.org/wiki/xacro">
+      <!-- The following values are approximate, and the camera node
+   publishing TF values with actual calibrated camera extrinsic values -->
+  <xacro:property name="d435_cam_depth_to_left_ir_offset" value="0.0"/>
+  <xacro:property name="d435_cam_depth_to_right_ir_offset" value="-0.050"/>
+  <xacro:property name="d435_cam_depth_to_color_offset" value="0.015"/>
+  <!-- The following values model the aluminum peripherial case for the
+    D435 camera, with the camera joint represented by the actual
+    peripherial camera tripod mount -->
+  <xacro:property name="d435_cam_width" value="0.090"/>
+  <xacro:property name="d435_cam_height" value="0.025"/>
+  <xacro:property name="d435_cam_depth" value="0.02505"/>
+  <xacro:property name="d435_cam_mount_from_center_offset" value="0.0149"/>
+  <!-- The following offset is relative the the physical D435 camera peripherial
+    camera tripod mount -->
+  <xacro:property name="d435_cam_depth_px" value="${d435_cam_mount_from_center_offset}"/>
+  <xacro:property name="d435_cam_depth_py" value="0.0175"/>
+  <xacro:property name="d435_cam_depth_pz" value="${d435_cam_height/2}"/>
+  <material name="Aluminum">
+    <color rgba="0.5 0.5 0.5 1"/>
+  </material>
     <joint name="intel_d435_mount_fixed" type="fixed">
         <origin xyz="${INTEL_D435_MOUNT_X} ${INTEL_D435_MOUNT_Y} ${INTEL_D435_MOUNT_Z}"
@@ -7,126 +27,120 @@
         <child link="camera_link"/>
     </joint>
-    <!-- camera depth joints and links -->
     <link name="camera_link">
-        <inertial>
-            <origin xyz="0 0 0" rpy="0 0 0"/>
-            <mass value="0.0446256012085417"/>
-            <inertia
-                    ixx="2.62358816469287E-05"
-                    ixy="3.51148589025883E-07"
-                    ixz="3.91275343984781E-11"
-                    iyy="4.02618646244092E-06"
-                    iyz="-6.05255657169474E-09"
-                    izz="2.64982132448102E-05"/>
-        </inertial>
-        <visual>
-            <origin xyz="0 0 0" rpy="0 0 0"/>
-            <geometry>
-                <mesh filename="package://infi_sim_v1/models/OPTIMUS_robot_001/meshes/intel_d435.stl" scale="1 1 1"/>
-            </geometry>
-            <material name="">
-                <color rgba="0.792156862745098 0.819607843137255 0.933333333333333 1"/>
-            </material>
-        </visual>
-        <collision>
-            <origin xyz="0 0 0" rpy="0 0 0"/>
-            <geometry>
-                <mesh filename="package://infi_sim_v1/models/OPTIMUS_robot_001/meshes/intel_d435.stl" scale="1 1 1"/>
-            </geometry>
-        </collision>
+      <visual>
+      <origin xyz="${d435_cam_mount_from_center_offset} 0.0 ${d435_cam_height/2}" rpy="${M_PI/2} 0 ${M_PI/2}"/>
+        <geometry>
+          <!-- <box size="${d435_cam_width} ${d435_cam_height} ${d435_cam_depth}"/> -->
+	      <mesh filename="package://infi_sim_v1/models/OPTIMUS_robot_001/meshes/d435.dae" />
+        </geometry>
+        <material name="Aluminum"/>
+      </visual>
+      <collision>
+        <origin xyz="0.0 0.0 ${d435_cam_height/2}" rpy="0 0 0"/>
+        <geometry>
+          <box size="${d435_cam_depth} ${d435_cam_width} ${d435_cam_height}"/>
+        </geometry>
+      </collision>
+      <inertial>
+        <!-- The following are not reliable values, and should not be used for modeling -->
+        <mass value="0.564" />
+        <origin xyz="0 0 0" />
+        <inertia ixx="0.003881243" ixy="0.0" ixz="0.0" iyy="0.000498940" iyz="0.0" izz="0.003879257" />
+      </inertial>
     </link>
+    <!--The following links will be not modeled and displayed.-->
+      <!-- camera depth joints and links -->
+      <joint name="camera_depth_joint" type="fixed">
+        <origin xyz="${d435_cam_depth_px} ${d435_cam_depth_py} ${d435_cam_depth_pz}" rpy="0 0 0"/>
+        <parent link="camera_link"/>
+        <child link="camera_depth_frame" />
+      </joint>
+      <link name="camera_depth_frame"/>
+      <joint name="camera_depth_optical_joint" type="fixed">
+        <origin xyz="0 0 0" rpy="${-M_PI/2} 0 ${-M_PI/2}" />
+        <parent link="camera_depth_frame" />
+        <child link="camera_depth_optical_frame" />
+      </joint>
+      <link name="camera_depth_optical_frame"/>
+      <!-- camera left IR joints and links -->
+      <joint name="camera_left_ir_joint" type="fixed">
+        <origin xyz="0 ${d435_cam_depth_to_left_ir_offset} 0" rpy="0 0 0" />
+        <parent link="camera_depth_frame" />
+        <child link="camera_left_ir_frame" />
+      </joint>
+      <link name="camera_left_ir_frame"/>
+      <joint name="camera_left_ir_optical_joint" type="fixed">
+        <origin xyz="0 0 0" rpy="${-M_PI/2} 0 ${-M_PI/2}" />
+        <parent link="camera_left_ir_frame" />
+        <child link="camera_left_ir_optical_frame" />
+      </joint>
+      <link name="camera_left_ir_optical_frame"/>
+      <!-- camera right IR joints and links -->
+      <joint name="camera_right_ir_joint" type="fixed">
+        <origin xyz="0 ${d435_cam_depth_to_right_ir_offset} 0" rpy="0 0 0" />
+        <parent link="camera_depth_frame" />
+        <child link="camera_right_ir_frame" />
+      </joint>
+      <link name="camera_right_ir_frame"/>
+      <joint name="camera_right_ir_optical_joint" type="fixed">
+        <origin xyz="0 0 0" rpy="${-M_PI/2} 0 ${-M_PI/2}" />
+        <parent link="camera_right_ir_frame" />
+        <child link="camera_right_ir_optical_frame" />
+      </joint>
+      <link name="camera_right_ir_optical_frame"/>
+      <!-- camera color joints and links -->
+      <joint name="camera_color_joint" type="fixed">
+        <origin xyz="0 ${d435_cam_depth_to_color_offset} 0" rpy="0 0 0" />
+        <parent link="camera_depth_frame" />
+        <child link="camera_color_frame" />
+      </joint>
+      <link name="camera_color_frame"/>
+      <joint name="camera_color_optical_joint" type="fixed">
+        <origin xyz="0 0 0" rpy="${-M_PI/2} 0 ${-M_PI/2}" />
+        <parent link="camera_color_frame" />
+        <child link="camera_color_optical_frame" />
+      </joint>
+      <link name="camera_color_optical_frame"/>
     <gazebo reference="camera_link">
-        <sensor type="depth" name="intel_d435">
-            <!--<pose>0 0 0 0 0 0</pose>-->
-            <always_on>1</always_on>
-            <visualize>true</visualize>
+      <sensor type="depth" name="camera">
+            <always_on>true</always_on>
+            <update_rate>20.0</update_rate>
             <camera>
-                <horizontal_fov>1.592</horizontal_fov>
-                <image>
-                    <width>1280</width>
-                    <height>800</height>
-                    <format>B8G8R8</format>
-                </image>
-                <depth_camera/>
-                <clip>
-                    <near>0.1</near>
-                    <far>100</far>
-                </clip>
+              <horizontal_fov>1.0471975512</horizontal_fov>
+              <image>
+                <format>R8G8B8</format>
+                <width>1280</width>
+                <height>800</height>
+              </image>
+              <clip>
+                <near>0.05</near>
+                <far>8.0</far>
+              </clip>
             </camera>
-            <plugin name="camera_controller" filename="libgazebo_ros_openni_kinect.so">
-                <alwaysOn>true</alwaysOn>
-                <updateRate>10.0</updateRate>
-                <cameraName>intel_d435/camera</cameraName>
-                <frameName>camera_link</frameName>
-                <imageTopicName>color/image_raw</imageTopicName>
-                <depthImageTopicName>depth/color/image_raw</depthImageTopicName>
-                <pointCloudTopicName>depth/color/points</pointCloudTopicName>
-                <cameraInfoTopicName>color/camera_info</cameraInfoTopicName>
-                <depthImageCameraInfoTopicName>depth/camera_info</depthImageCameraInfoTopicName>
-                <pointCloudCutoff>0.4</pointCloudCutoff>
-                <hackBaseline>0.07</hackBaseline>
-                <distortionK1>0.0</distortionK1>
-                <distortionK2>0.0</distortionK2>
-                <distortionK3>0.0</distortionK3>
-                <distortionT1>0.0</distortionT1>
-                <distortionT2>0.0</distortionT2>
-                <CxPrime>0.0</CxPrime>
-                <Cx>0.0</Cx>
-                <Cy>0.0</Cy>
-                <focalLength>0.0</focalLength>
+            <plugin name="kinect_camera_controller" filename="libgazebo_ros_openni_kinect.so">
+              <robotNamespace>/</robotNamespace>
+              <cameraName>camera</cameraName>
+              <alwaysOn>true</alwaysOn>
+              <updateRate>10</updateRate>
+              <imageTopicName>rgb/image_raw</imageTopicName>
+              <depthImageTopicName>depth/image_raw</depthImageTopicName>
+              <pointCloudTopicName>depth/points</pointCloudTopicName>
+              <cameraInfoTopicName>rgb/camera_info</cameraInfoTopicName>
+              <depthImageCameraInfoTopicName>depth/camera_info</depthImageCameraInfoTopicName>
+              <frameName>camera_depth_optical_frame</frameName>
+              <baseline>0.1</baseline>
+              <pointCloudCutoff>0.4</pointCloudCutoff>
+              <distortionK1>0.00000001</distortionK1>
+              <distortionK2>0.00000001</distortionK2>
+              <distortionK3>0.00000001</distortionK3>
+              <distortionT1>0.00000001</distortionT1>
+              <distortionT2>0.00000001</distortionT2>
+              <CxPrime>0</CxPrime>
+              <Cx>0</Cx>
+              <Cy>0</Cy>
+              <focalLength>0</focalLength>
+             <hackBaseline>0</hackBaseline>
             </plugin>
-        </sensor>
+          </sensor>
     </gazebo>
-    <!-- camera depth joints and links -->
-    <joint name="camera_depth_joint" type="fixed">
-        <origin xyz="0 -0.0122 0" rpy="0 0 0"/>
-        <parent link="camera_link"/>
-        <child link="camera_depth_frame"/>
-    </joint>
-    <link name="camera_depth_frame"/>
-    <joint name="camera_depth_optical_joint" type="fixed">
-        <origin xyz="0 0 0" rpy="${-M_PI/2} 0 ${-M_PI/2}"/>
-        <parent link="camera_depth_frame"/>
-        <child link="camera_depth_optical_frame"/>
-    </joint>
-    <link name="camera_depth_optical_frame"/>
-    <!-- camera left IR joints and links -->
-    <joint name="camera_left_ir_joint" type="fixed">
-        <origin xyz="0 -0.0322 0" rpy="0 0 0"/>
-        <parent link="camera_link"/>
-        <child link="camera_left_ir_frame"/>
-    </joint>
-    <link name="camera_left_ir_frame"/>
-    <joint name="camera_left_ir_optical_joint" type="fixed">
-        <origin xyz="0 0 0" rpy="${-M_PI/2} 0 ${-M_PI/2}"/>
-        <parent link="camera_left_ir_frame"/>
-        <child link="camera_left_ir_optical_frame"/>
-    </joint>
-    <link name="camera_left_ir_optical_frame"/>
-    <!-- camera right IR joints and links -->
-    <joint name="camera_right_ir_joint" type="fixed">
-        <origin xyz="0 0.0178 0" rpy="0 0 0"/>
-        <parent link="camera_link"/>
-        <child link="camera_right_ir_frame"/>
-    </joint>
-    <link name="camera_right_ir_frame"/>
-    <joint name="camera_right_ir_optical_joint" type="fixed">
-        <origin xyz="0 0 0" rpy="${-M_PI/2} 0 ${-M_PI/2}"/>
-        <parent link="camera_right_ir_frame"/>
-        <child link="camera_right_ir_optical_frame"/>
-    </joint>
-    <link name="camera_right_ir_optical_frame"/>
-    <!-- camera fisheye joints and links -->
-    <joint name="camera_fisheye_joint" type="fixed">
-        <origin xyz="0 0.0322 0" rpy="0 0 0"/>
-        <parent link="camera_link"/>
-        <child link="camera_fisheye_frame"/>
-    </joint>
-    <link name="camera_fisheye_frame"/>
-    <joint name="camera_fisheye_optical_joint" type="fixed">
-        <origin xyz="0 0 0" rpy="${-M_PI/2} 0 ${-M_PI/2}"/>
-        <parent link="camera_fisheye_frame"/>
-        <child link="camera_fisheye_optical_frame"/>
-    </joint>
-    <link name="camera_fisheye_optical_frame"/>
 </robot>

Commit message: with depth cam

File: infi_sim_v1/models/OPTIMUS_robot_001/model-no-arm.xacro (robot description, xacro)
@@ -3,9 +3,4 @@
     <xacro:property name="deg_to_rad" value="0.01745329251994329577"/>
     <xacro:property name="camera_link" value="0.05" /> <!-- Size of square 'camera' box -->
-    <!--xacro:include filename="sensors/xtion_pro_live.urdf.xacro"/-->
-    <!--xacro:xtion_pro_live name="rgbd_camera" parent="end">
-        <origin xyz="0 0 0.1" rpy="0 0 0"/>
-        <origin xyz="0 0 0.1" rpy="${-90.0 * deg_to_rad} 0 ${-90.0 * deg_to_rad}"/>
-    </xacro:xtion_pro_live-->
     <xacro:property name="INTEL_D435_MOUNT_LINK" value="camera_mount_dummy_link"/>
     <xacro:property name="INTEL_D435_MOUNT_X" value="0.1"/>
@@ -16,5 +11,4 @@
     <xacro:property name="INTEL_D435_MOUNT_Y" value="${M_PI*0.0}"/>
     <xacro:include filename="sensors/intel_d435.xacro"/>
-    <!--xacro:include filename="sensors/intel_cam.xacro" name="camera_link" ros_topic="/d435"/-->
     <link name="base_footprint"/>
     <joint name="base_footprint_joint" type="fixed">

File: infi_sim_v1/models/OPTIMUS_robot_001/model.xacro (robot description, xacro)
@@ -8,11 +8,4 @@
     <xacro:property name="MANIPULATOR_MOUNT_Z" value="0.0"/>
     <xacro:include filename="manipulator_h.xacro"/>
-    <!--xacro:include filename="sensors/xtion_pro_live.urdf.xacro"/-->
-    <!--xacro:xtion_pro_live name="rgbd_camera" parent="end">
-        <origin xyz="0 0 0.1" rpy="0 0 0"/-->
-        <!--origin xyz="0 0 0.1" rpy="${-90.0 * deg_to_rad} 0 ${-90.0 * deg_to_rad}"/-->
-        <!--<origin xyz="0 0 0.1" rpy="0 ${75.0 * deg_to_rad} 0"/>-->
-        <!--<optical_origin xyz="0 0 0.1" rpy="${-90.0 * deg_to_rad} 0 ${-90.0 * deg_to_rad}"/>-->
-    <!--/xacro:xtion_pro_live-->
     <xacro:property name="INTEL_D435_MOUNT_LINK" value="camera_mount_dummy_link"/>
     <xacro:property name="INTEL_D435_MOUNT_X" value="0.1"/>
@@ -22,6 +15,5 @@
     <xacro:property name="INTEL_D435_MOUNT_P" value="${M_PI*0.0}"/>
     <xacro:property name="INTEL_D435_MOUNT_Y" value="${M_PI*0.0}"/>
-    <!--<xacro:include filename="sensors/intel_d435.xacro"/>-->
-    <!--    <xacro:include filename="sensors/intel_cam.xacro" name="camera_link" ros_topic="/d435"/>-->
+    <xacro:include filename="sensors/intel_d435.xacro"/>
     <link name="base_footprint"/>
     <joint name="base_footprint_joint" type="fixed">

Commit message: fix lidar location

File: infi_sim_v1/models/OPTIMUS_robot_001/model-no-arm.xacro (robot description, xacro)
@@ -284,5 +284,5 @@
         <parent link="base_link"/>
         <child link="ray_sensor_front"/>
-        <origin xyz="0.5 0 0.5" rpy="0 0 0"/>
+        <origin xyz="0.65 0 0.120" rpy="0 0 0"/>
         <axis xyz="0 0 1"/>
     </joint>

File: infi_sim_v1/models/OPTIMUS_robot_001/model.xacro (robot description, xacro)
@@ -290,5 +290,5 @@
         <parent link="base_link"/>
         <child link="ray_sensor_front"/>
-        <origin xyz="0.5 0 0.5" rpy="0 0 0"/>
+        <origin xyz="0.65 0 0.120" rpy="0 0 0"/>
         <axis xyz="0 0 1"/>
     </joint>

Commit message: Merge remote-tracking branch 'origin/master'

File: infi_sim_v1/models/OPTIMUS_robot_001/model-no-arm.xacro (robot description, xacro)
@@ -3,9 +3,4 @@
     <xacro:property name="deg_to_rad" value="0.01745329251994329577"/>
     <xacro:property name="camera_link" value="0.05" /> <!-- Size of square 'camera' box -->
-    <!--xacro:include filename="sensors/xtion_pro_live.urdf.xacro"/-->
-    <!--xacro:xtion_pro_live name="rgbd_camera" parent="end">
-        <origin xyz="0 0 0.1" rpy="0 0 0"/>
-        <origin xyz="0 0 0.1" rpy="${-90.0 * deg_to_rad} 0 ${-90.0 * deg_to_rad}"/>
-    </xacro:xtion_pro_live-->
     <xacro:property name="INTEL_D435_MOUNT_LINK" value="camera_mount_dummy_link"/>
     <xacro:property name="INTEL_D435_MOUNT_X" value="0.1"/>
@@ -15,6 +10,5 @@
     <xacro:property name="INTEL_D435_MOUNT_P" value="${M_PI*0.0}"/>
     <xacro:property name="INTEL_D435_MOUNT_Y" value="${M_PI*0.0}"/>
-    <!--xacro:include filename="sensors/intel_d435.xacro"/-->
-    <!--xacro:include filename="sensors/intel_cam.xacro" name="camera_link" ros_topic="/d435"/-->
+    <xacro:include filename="sensors/intel_d435.xacro"/>
     <link name="base_footprint"/>
     <joint name="base_footprint_joint" type="fixed">

Commit message: CNC coliision simplified

File: infi_sim_v1/models/OPTIMUS_robot_001/model-no-arm.xacro (robot description, xacro)
@@ -284,5 +284,5 @@
         <parent link="base_link"/>
         <child link="ray_sensor_front"/>
-        <origin xyz="0.65 0 0.120" rpy="0 0 0"/>
+        <origin xyz="0.8 0 0.120" rpy="0 0 0"/>
         <axis xyz="0 0 1"/>
     </joint>

File: infi_sim_v1/models/OPTIMUS_robot_001/model.xacro (robot description, xacro)
@@ -290,5 +290,5 @@
         <parent link="base_link"/>
         <child link="ray_sensor_front"/>
-        <origin xyz="0.65 0 0.120" rpy="0 0 0"/>
+        <origin xyz="0.7 0 0.120" rpy="0 0 0"/>
         <axis xyz="0 0 1"/>
     </joint>
